File: templates/IO30/io30.kicad_sch (KiCad schematic)
At the start: 1 part, among them J101 CONN HDR 30POS 2.54 R/A

Commit message: template: IO30
Other:
- note added: "100mA max"
Changed lines of the file:
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@@
+		)
+	)
+	(text "100mA max"
+		(exclude_from_sim no)
+		(at 95.758 110.49 0)
+		(effects
+			(font
+				(size 1 1)
+				(color 132 132 132 1)
+			)
+			(justify left bottom)
+		)
+	)
+	(text "100mA max"
+		(exclude_from_sim no)
+		(at 95.25 146.05 0)
+		(effects
+			(font
+				(size 1 1)
+				(color 132 132 132 1)
+			)
+			(justify left bottom)
 		)
 	)
