File: templates/Vhrd Default/default_vhrd.kicad_pcb (KiCad board)
At the start: 4 copper layers, 12 parts

Commit message: template: io30
Parts:
- renumbered V1901 to V201, V1908 to V202, V1903 to V203, V1902 to V204, V1910 to V205, V1904 to V206, V1909 to V207, V1906 to V208, V1905 to V209, V1907 to V210, V1911 to V211, V1912 to V212
Changed lines of the file:
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@@
 		(layer "F.Cu")
 		(at 197.6 150.3)
-		(property "Reference" "V1907"
+		(property "Reference" "V210"
 			(at 0 -0.5 0)
 			(unlocked yes)
@@
 		(layer "F.Cu")
 		(at 205.85 150.3)
-		(property "Reference" "V1905"
+		(property "Reference" "V209"
 			(at 0 -0.5 0)
 			(unlocked yes)
@@
 		(layer "F.Cu")
 		(at 245.4 151.6)
-		(property "Reference" "V1901"
+		(property "Reference" "V201"
 			(at 2 -5.75 0)
 			(unlocked yes)
@@
 		(descr "KiCad Logo")
 		(tags "Logo KiCad")
-		(property "Reference" "V1908"
+		(property "Reference" "V202"
 			(at 0 -5.08 0)
 			(layer "F.SilkS")
@@
 		(layer "F.Cu")
 		(at 177.3 149.5)
-		(property "Reference" "V1909"
+		(property "Reference" "V207"
 			(at 0 -0.5 0)
 			(unlocked yes)
@@
 		(layer "F.Cu")
 		(at 220.1 148.65)
-		(property "Reference" "V1902"
+		(property "Reference" "V204"
 			(at 2 -5.75 0)
 			(unlocked yes)
@@
 		(descr "Waste Electrical and Electronic Equipment Directive https://eur-lex.europa.eu/legal-content/EN/TXT/PDF/?uri=CELEX:32012L0019#page=29")
 		(tags "Logo WEEE")
-		(property "Reference" "V1910"
+		(property "Reference" "V205"
 			(at 0 0 0)
 			(layer "F.SilkS")
@@
 		(layer "F.Cu")
 		(at 256.2 149.5)
-		(property "Reference" "V1912"
+		(property "Reference" "V212"
 			(at 0 -0.5 0)
 			(unlocked yes)
@@
 		(layer "B.Cu")
 		(at 225.5 163.1)
-		(property "Reference" "V1903"
+		(property "Reference" "V203"
 			(at 0 0.5 180)
 			(unlocked yes)
@@
 		(layer "B.Cu")
 		(at 215.2 160.3)
-		(property "Reference" "V1906"
+		(property "Reference" "V208"
 			(at 0 0.5 180)
 			(unlocked yes)
@@
 		(layer "B.Cu")
 		(at 204.8 150.3 180)
-		(property "Reference" "V1904"
+		(property "Reference" "V206"
 			(at 0 0.5 0)
 			(unlocked yes)
@@
 		(layer "B.Cu")
 		(at 192.5 149.5 180)
-		(property "Reference" "V1911"
+		(property "Reference" "V211"
 			(at 0 0.5 0)
 			(unlocked yes)

Commit message: RoHS symbol
Parts:
- added V213: RoHS, vhrd_visual:RoHS-Logo_6mm_SilkScreen, F.Cu at (200.3, 159.5)
- moved V205 11.9 mm to (187.7, 160.4)
- moved V202 10.5 mm to (174.6, 159.6)
