File: templates/Vhrd Default/mechanical.kicad_sch (KiCad schematic)
At the start: 12 parts

Commit message: template: io30
Parts:
- renumbered V1901 to V201, V1908 to V202, V1903 to V203, V1902 to V204, V1910 to V205, V1904 to V206, V1909 to V207, V1906 to V208, V1905 to V209, V1907 to V210, V1911 to V211, V1912 to V212
Changed lines of the file:
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@@
 		(in_pos_files yes)
 		(dnp no)
-		(property "Reference" "V1901"
+		(property "Reference" "V201"
 			(at 30.48 31.75 0)
 			(show_name no)
@@
 			(project "default_vhrd"
 				(path "/40f6bb79-f555-4b81-9ba4-c7b6659be11e/e8024289-d464-4f5f-b671-8fa26c9108fa"
-					(reference "V1901")
+					(reference "V201")
 					(unit 1)
 				)
@@
 		(in_pos_files yes)
 		(dnp no)
-		(property "Reference" "V1909"
+		(property "Reference" "V207"
 			(at 88.9 64.77 0)
 			(show_name no)
@@
 			(project "default_vhrd"
 				(path "/40f6bb79-f555-4b81-9ba4-c7b6659be11e/e8024289-d464-4f5f-b671-8fa26c9108fa"
-					(reference "V1909")
+					(reference "V207")
 					(unit 1)
 				)
@@
 		(in_pos_files yes)
 		(dnp no)
-		(property "Reference" "V1906"
+		(property "Reference" "V208"
 			(at 82.55 120.65 0)
 			(show_name no)
@@
 			(project "default_vhrd"
 				(path "/40f6bb79-f555-4b81-9ba4-c7b6659be11e/e8024289-d464-4f5f-b671-8fa26c9108fa"
-					(reference "V1906")
+					(reference "V208")
 					(unit 1)
 				)
@@
 		(in_pos_files yes)
 		(dnp no)
-		(property "Reference" "V1904"
+		(property "Reference" "V206"
 			(at 85.09 31.75 0)
 			(show_name no)
@@
 			(project "default_vhrd"
 				(path "/40f6bb79-f555-4b81-9ba4-c7b6659be11e/e8024289-d464-4f5f-b671-8fa26c9108fa"
-					(reference "V1904")
+					(reference "V206")
 					(unit 1)
 				)
@@
 		(in_pos_files yes)
 		(dnp no)
-		(property "Reference" "V1907"
+		(property "Reference" "V210"
 			(at 110.49 31.75 0)
 			(show_name no)
@@
 			(project "default_vhrd"
 				(path "/40f6bb79-f555-4b81-9ba4-c7b6659be11e/e8024289-d464-4f5f-b671-8fa26c9108fa"
-					(reference "V1907")
+					(reference "V210")
 					(unit 1)
 				)
@@
 		(in_pos_files yes)
 		(dnp no)
-		(property "Reference" "V1911"
+		(property "Reference" "V211"
 			(at 107.95 64.77 0)
 			(show_name no)
@@
 			(project "default_vhrd"
 				(path "/40f6bb79-f555-4b81-9ba4-c7b6659be11e/e8024289-d464-4f5f-b671-8fa26c9108fa"
-					(reference "V1911")
+					(reference "V211")
 					(unit 1)
 				)
@@
 		(in_pos_files yes)
 		(dnp no)
-		(property "Reference" "#PWR01901"
+		(property "Reference" "#PWR0201"
 			(at 25.4 48.26 0)
 			(hide yes)
@@
 			(project "default_vhrd"
 				(path "/40f6bb79-f555-4b81-9ba4-c7b6659be11e/e8024289-d464-4f5f-b671-8fa26c9108fa"
-					(reference "#PWR01901")
+					(reference "#PWR0201")
 					(unit 1)
 				)
@@
 		(in_pos_files yes)
 		(dnp no)
-		(property "Reference" "V1910"
+		(property "Reference" "V205"
 			(at 55.88 120.65 0)
 			(show_name no)
@@
 			(project "default_vhrd"
 				(path "/40f6bb79-f555-4b81-9ba4-c7b6659be11e/e8024289-d464-4f5f-b671-8fa26c9108fa"
-					(reference "V1910")
+					(reference "V205")
 					(unit 1)
 				)
@@
 		(in_pos_files yes)
 		(dnp no)
-		(property "Reference" "V1905"
+		(property "Reference" "V209"
 			(at 95.25 96.52 0)
 			(show_name no)
@@
 			(project "default_vhrd"
 				(path "/40f6bb79-f555-4b81-9ba4-c7b6659be11e/e8024289-d464-4f5f-b671-8fa26c9108fa"
-					(reference "V1905")
+					(reference "V209")
 					(unit 1)
 				)
@@
 		(dnp no)
 		(fields_autoplaced yes)
-		(property "Reference" "V1912"
+		(property "Reference" "V212"
 			(at 124.46 125.7299 0)
 			(show_name no)
@@
 			(project "default_vhrd"
 				(path "/40f6bb79-f555-4b81-9ba4-c7b6659be11e/e8024289-d464-4f5f-b671-8fa26c9108fa"
-					(reference "V1912")
+					(reference "V212")
 					(unit 1)
 				)
@@
 		(in_pos_files yes)
 		(dnp no)
-		(property "Reference" "V1903"
+		(property "Reference" "V203"
 			(at 43.18 64.77 0)
 			(show_name no)
@@
 			(project "default_vhrd"
 				(path "/40f6bb79-f555-4b81-9ba4-c7b6659be11e/e8024289-d464-4f5f-b671-8fa26c9108fa"
-					(reference "V1903")
+					(reference "V203")
 					(unit 1)
 				)
@@
 		(in_pos_files yes)
 		(dnp no)
-		(property "Reference" "V1902"
+		(property "Reference" "V204"
 			(at 55.88 31.75 0)
 			(show_name no)
@@
 			(project "default_vhrd"
 				(path "/40f6bb79-f555-4b81-9ba4-c7b6659be11e/e8024289-d464-4f5f-b671-8fa26c9108fa"
-					(reference "V1902")
+					(reference "V204")
 					(unit 1)
 				)
@@
 		(in_pos_files yes)
 		(dnp no)
-		(property "Reference" "V1908"
+		(property "Reference" "V202"
 			(at 33.02 120.65 0)
 			(show_name no)
@@
 			(project "default_vhrd"
 				(path "/40f6bb79-f555-4b81-9ba4-c7b6659be11e/e8024289-d464-4f5f-b671-8fa26c9108fa"
-					(reference "V1908")
-					(unit 1)
-				)
+					(reference "V202")
+					(unit 1)
+				)

Commit message: RoHS symbol
Parts:
- added V213: RoHS, vhrd_visual:RoHS-Logo_6mm_SilkScreen, symbol vhrd_visual:SYM
Changed lines of the file:
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@@
+	)
+	(symbol
+		(lib_id "vhrd_visual:SYM")
+		(at 30.48 138.43 0)
+		(unit 1)
+		(body_style 1)
+		(exclude_from_sim no)
+		(in_bom no)
+		(on_board yes)
+		(in_pos_files yes)
+		(dnp no)
+		(property "Reference" "V213"
+			(at 30.48 137.16 0)
+			(show_name no)
+			(do_not_autoplace no)
+			(effects
+				(font
+					(size 1.27 1.27)
+				)
+				(justify left)
+			)
+		)
+		(property "Value" "RoHS"
+			(at 40.64 147.32 0)
+			(show_name no)
+			(do_not_autoplace no)
+			(effects
+				(font
+					(size 1.27 1.27)
+				)
+				(justify left)
+			)
+		)
+		(property "Footprint" "vhrd_visual:RoHS-Logo_6mm_SilkScreen"
+			(at 38.1 147.32 0)
+			(hide yes)
+			(show_name no)
+			(do_not_autoplace no)
+			(effects
+				(font
+					(size 1.27 1.27)
+				)
+			)
+		)
+		(property "Datasheet" ""
+			(at 30.48 138.43 0)
+			(hide yes)
+			(show_name no)
+			(do_not_autoplace no)
+			(effects
+				(font
+					(size 1.27 1.27)
+				)
+			)
+		)
+		(property "Description" ""
+			(at 30.48 138.43 0)
+			(hide yes)
+			(show_name no)
+			(do_not_autoplace no)
+			(effects
+				(font
+					(size 1.27 1.27)
+				)
+			)
+		)
+		(property "Iworking" ""
+			(at 30.48 138.43 0)
+			(hide yes)
+			(show_name no)
+			(do_not_autoplace no)
+			(effects
+				(font
+					(size 1.27 1.27)
+				)
+			)
+		)
+		(instances
+			(project "default_vhrd"
+				(path "/40f6bb79-f555-4b81-9ba4-c7b6659be11e/e8024289-d464-4f5f-b671-8fa26c9108fa"
+					(reference "V213")
+					(unit 1)
+				)
+			)
+		)
 	)
 	(symbol
